File: eagle-design/main.brd (EAGLE design)
At the start: 132.1 x 33.3 mm, 16 parts, among them IC1 7805T

Commit message: Added new code
Parts:
- added R5, R6: 10K, adafruit:0805-THM
- moved R3 5.47 mm to (54.4, 23.2)
- moved R2 3.69 mm to (54.3, 18.7)
- moved R1 2.21 mm to (54.0, 14.0)
- moved R4 1.52 mm to (54.5, 6.93)
Connections:
- new net VCC: R5.1, R6.1
- net N$7: now also R6.2
- net N$8: now also R5.2
Routing:
- net N$32: track 106.1 -> 101.6 mm
- net N$6: track 29.7 -> 32.2 mm
- net N$2: track 5.08 -> 7.17 mm
- net N$5: track 32.1 -> 34.1 mm
- net N$11: track 71.1 -> 72.6 mm
Other:
- outline, holes or cut-outs redrawn

Commit message: Added updated eagle design
Parts:
- moved R1 2.35 mm to (55.6, 15.8)
- moved R2 1.94 mm to (55.7, 20.0)
- moved R3 1.64 mm to (55.7, 24.2)
- moved R5 1.17 mm to (55.8, 32.4)
- moved R6 0.83 mm to (55.7, 28.5)
- moved R4 0.43 mm to (54.1, 7.14)
- moved LED1 0.33 mm to (43.9, 28.9)
Connections:
- removed net VCC: R5.1, R6.1
- net N$14: now also R5.1, R6.1
Routing:
- net N$14: track 53.4 -> 96.6 mm
- net N$7: track 64.4 -> 84.0 mm
- net N$8: track 72.8 -> 88.5 mm
- net N$5: track 34.1 -> 31.7 mm
- net N$6: track 32.2 -> 30.2 mm
- net N$32: track 101.6 -> 102.6 mm
- net N$3: track 5.56 -> 6.48 mm
- net N$4: track 4.59 -> 5.48 mm
- net 0: track 226.2 -> 227.0 mm
Other:
- board text added: "3.3V"
- board text removed: "VCC"
- board text removed: "Vcc"

Commit message: Added new design and export image
Parts:
- moved R4 1.38 mm to (55.5, 7.24)
Routing:
- net N$32: track 102.6 -> 100.6 mm
- net N$13: track 11.9 -> 12.5 mm
Changed lines of the file:
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@@
 <text x="55.88" y="17.526" size="1.016" layer="21">220 Ω</text>
 <text x="55.9308" y="13.3604" size="1.016" layer="21">220 Ω</text>
-<text x="52.2986" y="4.7498" size="1.016" layer="21">10K Ω</text>
+<text x="53.3908" y="4.7752" size="1.016" layer="21">10K Ω</text>
 <text x="121.285" y="24.13" size="1.778" layer="21">BMP280</text>
 <text x="117.475" y="10.16" size="1.778" layer="21">DHT22</text>
@@
 <wire x1="35.56" y1="33.02" x2="35.56" y2="34.29" width="0.3556" layer="22"/>
 <wire x1="35.56" y1="34.29" x2="34.925" y2="34.925" width="0.3556" layer="22"/>
-<wire x1="66.675" y1="31.115" x2="66.675" y2="5.715" width="0.1524" layer="21"/>
-<wire x1="66.675" y1="5.715" x2="114.935" y2="5.715" width="0.1524" layer="21"/>
-<wire x1="114.935" y1="5.715" x2="114.935" y2="31.115" width="0.1524" layer="21"/>
-<wire x1="114.935" y1="31.115" x2="66.675" y2="31.115" width="0.1524" layer="21"/>
+<wire x1="66.675" y1="31.3182" x2="66.675" y2="5.2578" width="0.1524" layer="21"/>
+<wire x1="66.675" y1="5.2578" x2="114.935" y2="5.2578" width="0.1524" layer="21"/>
+<wire x1="114.935" y1="5.2578" x2="114.935" y2="31.3182" width="0.1524" layer="21"/>
+<wire x1="114.935" y1="31.3182" x2="66.675" y2="31.3182" width="0.1524" layer="21"/>
 <text x="55.9562" y="26.0096" size="1.016" layer="21">10K Ω</text>
 <text x="56.0324" y="29.9974" size="1.016" layer="21">10K Ω</text>
+<polygon width="0.0254" layer="17">
+<vertex x="24.7904" y="34.163"/>
+<vertex x="34.9504" y="34.163"/>
+<vertex x="34.9504" y="32.512"/>
+<vertex x="34.9758" y="32.512"/>
+<vertex x="34.9758" y="32.4866"/>
+<vertex x="34.036" y="32.4866"/>
+<vertex x="34.036" y="30.734"/>
+<vertex x="34.925" y="30.734"/>
+<vertex x="34.925" y="30.7086"/>
+<vertex x="34.925" y="27.4574"/>
+<vertex x="24.765" y="27.4574"/>
+<vertex x="24.765" y="30.734"/>
+<vertex x="24.8158" y="30.734"/>
+<vertex x="25.654" y="30.734"/>
+<vertex x="25.654" y="30.7594"/>
+<vertex x="25.654" y="32.4866"/>
+<vertex x="24.765" y="32.4866"/>
+<vertex x="24.765" y="34.163"/>
+</polygon>
+<polygon width="0.0254" layer="29">
+<vertex x="25.8572" y="33.909"/>
+<vertex x="33.8328" y="33.909"/>
+<vertex x="33.8328" y="27.6098"/>
+<vertex x="25.8572" y="27.6098"/>
+</polygon>
+<polygon width="0.0254" layer="30">
+<vertex x="25.8064" y="33.909"/>
+<vertex x="33.8074" y="33.909"/>
+<vertex x="33.8074" y="27.7368"/>
+<vertex x="25.8064" y="27.7368"/>
+</polygon>
 </plain>
 <attributes>
@@
 <elements>
 <element name="C3" library="adafruit" package="E2,5-6E" value="" x="9.525" y="10.795" smashed="yes">
-<attribute name="NAME" x="8.382" y="12.319" size="1.27" layer="25" ratio="10"/>
+<attribute name="NAME" x="11.176" y="13.7922" size="1.27" layer="25" ratio="10"/>
 <attribute name="VALUE" x="12.192" y="8.255" size="1.27" layer="27" ratio="10"/>
 </element>
 <element name="C4" library="adafruit" package="E2,5-6E" value="" x="17.145" y="10.795" smashed="yes" rot="R180">
-<attribute name="NAME" x="17.018" y="13.081" size="1.27" layer="25" ratio="10" rot="R180"/>
+<attribute name="NAME" x="21.336" y="14.3002" size="1.27" layer="25" ratio="10" rot="R180"/>
 <attribute name="VALUE" x="14.478" y="13.335" size="1.27" layer="27" ratio="10" rot="R180"/>
 </element>
@@
 <attribute name="VALUE" x="55.9244" y="21.6344" size="1.27" layer="27" ratio="10"/>
 </element>
-<element name="R4" library="adafruit" package="0805-THM" value="10K" x="54.102" y="7.1374" smashed="yes">
-<attribute name="NAME" x="52.1462" y="8.7884" size="1.27" layer="25" ratio="10"/>
-<attribute name="VALUE" x="55.0354" y="8.7312" size="1.27" layer="27" ratio="10"/>
+<element name="R4" library="adafruit" package="0805-THM" value="10K" x="55.4736" y="7.239" smashed="yes">
+<attribute name="NAME" x="53.5178" y="8.89" size="1.27" layer="25" ratio="10"/>
+<attribute name="VALUE" x="56.407" y="8.8328" size="1.27" layer="27" ratio="10"/>
 </element>
 <element name="S1" library="switch-omron" library_urn="urn:adsk.eagle:library:377" package="B3F-10XX" package3d_urn="urn:adsk.eagle:package:27496/1" value="" x="42.545" y="8.255" smashed="yes" rot="R180">
@@
 <wire x1="66.675" y1="4.445" x2="65.405" y2="5.715" width="0.3556" layer="1"/>
 <via x="65.405" y="5.715" extent="1-16" drill="0.35"/>
-<wire x1="65.405" y1="5.715" x2="63.9826" y2="7.1374" width="0.3556" layer="16"/>
-<wire x1="63.9826" y1="7.1374" x2="59.182" y2="7.1374" width="0.3556" layer="16"/>
+<wire x1="65.405" y1="5.715" x2="63.881" y2="7.239" width="0.3556" layer="16"/>
+<wire x1="63.881" y1="7.239" x2="60.5536" y2="7.239" width="0.3556" layer="16"/>
 <wire x1="60.7314" y1="24.2316" x2="62.1792" y2="22.7838" width="0.1524" layer="16"/>
 <wire x1="62.1792" y1="22.7838" x2="62.1792" y2="11.3792" width="0.1524" layer="16"/>
 <wire x1="62.1792" y1="11.3792" x2="61.595" y2="10.795" width="0.1524" layer="16"/>
-<wire x1="61.595" y1="10.795" x2="59.182" y2="8.382" width="0.3556" layer="16"/>
-<wire x1="59.182" y1="7.1374" x2="59.182" y2="8.382" width="0.3556" layer="16"/>
+<wire x1="61.595" y1="10.795" x2="60.5536" y2="9.7536" width="0.3556" layer="16"/>
+<wire x1="60.5536" y1="7.239" x2="60.5536" y2="9.7536" width="0.3556" layer="16"/>
 <wire x1="32.385" y1="15.875" x2="34.925" y2="13.335" width="0.3556" layer="16"/>
 <wire x1="42.545" y1="13.335" x2="43.9928" y2="11.8872" width="0.3556" layer="16"/>
@@
 <contactref element="R4" pad="1"/>
 <wire x1="47.0154" y1="10.5156" x2="45.7962" y2="10.5156" width="0.1524" layer="1"/>
-<wire x1="49.022" y1="7.1374" x2="49.022" y2="8.509" width="0.1524" layer="1"/>
-<wire x1="49.022" y1="8.509" x2="47.0154" y2="10.5156" width="0.1524" layer="1"/>
+<wire x1="50.3936" y1="7.239" x2="50.292" y2="7.239" width="0.1524" layer="1"/>
+<wire x1="50.292" y1="7.239" x2="47.0154" y2="10.5156" width="0.1524" layer="1"/>
 <wire x1="45.7962" y1="10.5156" x2="39.2938" y2="10.5156" width="0.1524" layer="1"/>
 </signal>
@@
 <wire x1="49.784" y1="29.337" x2="50.6476" y2="28.4734" width="0.1524" layer="16"/>
 </signal>
+<signal name="N$16">
+<via x="27.3558" y="32.7406" extent="1-16" drill="0.35"/>
+</signal>
+<signal name="N$17">
+<via x="26.8732" y="31.7246" extent="1-16" drill="0.35"/>
+</signal>
+<signal name="N$18">
+<via x="26.7716" y="30.7848" extent="1-16" drill="0.35"/>
+</signal>
+<signal name="N$19">
+<via x="27.1526" y="29.3624" extent="1-16" drill="0.35"/>
+</signal>
+<signal name="N$20">
+<via x="32.1818" y="32.893" extent="1-16" drill="0.35"/>
+</signal>
+<signal name="N$21">
+<via x="32.7914" y="31.9278" extent="1-16" drill="0.35"/>
+</signal>
+<signal name="N$22">
+<via x="32.893" y="30.5562" extent="1-16" drill="0.35"/>
+</signal>
+<signal name="N$23">
+<via x="32.4866" y="29.2608" extent="1-16" drill="0.35"/>
+</signal>
+<signal name="N$24">
+<via x="27.8638" y="28.4734" extent="1-16" drill="0.35"/>
+</signal>
+<signal name="N$25">
+<via x="31.6484" y="28.3718" extent="1-16" drill="0.35"/>
+</signal>
+<signal name="N$9">
+<via x="26.5938" y="33.2994" extent="1-16" drill="0.35"/>
+</signal>
+<signal name="N$15">
+<via x="33.1216" y="33.1978" extent="1-16" drill="0.35"/>
+</signal>
+<signal name="N$26">
+<via x="32.6898" y="28.2702" extent="1-16" drill="0.35"/>
+</signal>
+<signal name="N$27">
+<via x="26.6446" y="28.3464" extent="1-16" drill="0.35"/>
+</signal>
+<signal name="N$28">
+<via x="26.416" y="29.9212" extent="1-16" drill="0.35"/>
+</signal>
+<signal name="N$29">
+<via x="28.1432" y="33.401" extent="1-16" drill="0.35"/>
+</signal>
 </signals>
