File: eagle-design/info.sch (EAGLE design)
At the start: 17 parts

Commit message: Addedd new design
Other:
- note added: "SD Card Module (ESP)"
- note added: "SDCard Module (MEGA)"
- moved on the sheet: JP3, R7

Commit message: Added motherboard design and image exports
Parts:
- R1, R2, R3, R4, R5, R6, R7: value (none) -> 68
Changed lines of the file:
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@@
 <part name="LED6" library="adafruit" deviceset="LED" device="3MM"/>
 <part name="LED7" library="adafruit" deviceset="LED" device="3MM"/>
-<part name="R1" library="adafruit" deviceset="R-US_" device="0204/7"/>
-<part name="R2" library="adafruit" deviceset="R-US_" device="0204/7"/>
-<part name="R3" library="adafruit" deviceset="R-US_" device="0204/7"/>
-<part name="R4" library="adafruit" deviceset="R-US_" device="0204/7"/>
-<part name="R5" library="adafruit" deviceset="R-US_" device="0204/7"/>
-<part name="R6" library="adafruit" deviceset="R-US_" device="0204/7"/>
-<part name="R7" library="adafruit" deviceset="R-US_" device="0204/7"/>
+<part name="R1" library="adafruit" deviceset="R-US_" device="0204/7" value="68"/>
+<part name="R2" library="adafruit" deviceset="R-US_" device="0204/7" value="68"/>
+<part name="R3" library="adafruit" deviceset="R-US_" device="0204/7" value="68"/>
+<part name="R4" library="adafruit" deviceset="R-US_" device="0204/7" value="68"/>
+<part name="R5" library="adafruit" deviceset="R-US_" device="0204/7" value="68"/>
+<part name="R6" library="adafruit" deviceset="R-US_" device="0204/7" value="68"/>
+<part name="R7" library="adafruit" deviceset="R-US_" device="0204/7" value="68"/>
 <part name="JP3" library="adafruit" deviceset="PINHD-1X6" device=""/>
 <part name="JP4" library="adafruit" deviceset="PINHD-1X6" device=""/>
