File: eagle-design/board.brd (EAGLE design)
At the start: 160 x 100 mm, 23 parts, among them IC1 7805T

Commit message: Updated board design
Routing:
- net N$25: track 43.4 -> 48.4 mm, vias 0 -> 1
- net N$20: track 151.0 -> 152.3 mm
- net N$17: track 90.0 -> 91.2 mm
- net N$13: track 87.8 -> 88.6 mm
- net N$2: track 244.8 -> 244.1 mm
